File: Kicad/TeensyMonoSynth/TeensyMonoSynth.kicad_sch (KiCad schematic)
At the start: 22 parts, among them U1 74HCT4051, U2 74HCT4051, U3 74HCT4051

Commit message: add teensy symbol and footprint libs
Parts:
- RV1: footprint Potentiometer_THT:Potentiometer_Alps_RK09L_Single_Vertical -> teensy.pretty-master:Teensy30_31_32_LC
Changed lines of the file:
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@@
       (effects (font (size 1.27 1.27)) (justify right))
     )
-    (property "Footprint" "Potentiometer_THT:Potentiometer_Alps_RK09L_Single_Vertical" (at 38.1 25.4 0)
+    (property "Footprint" "teensy.pretty-master:Teensy30_31_32_LC" (at 38.1 25.4 0)
       (effects (font (size 1.27 1.27)) hide)
     )

Commit message: PCB LAYOUT COMPLETE
Parts:
- added D1, D2, D3: LED, LED_THT:LED_D3.0mm, symbol Device:LED
- added J1: Conn_01x16_Socket, Connector_IDC:IDC-Header_2x08_P2.54mm_Vertical, symbol Connector:Conn_01x16_Socket
- added R1, R2, R3: R, Resistor_THT:R_Axial_DIN0207_L6.3mm_D2.5mm_P10.16mm_Horizontal, symbol Device:R
- added SW1: SW_Push, Button_Switch_THT:SW_PUSH-12mm, symbol Switch:SW_Push
- RV1: footprint teensy.pretty-master:Teensy30_31_32_LC -> Potentiometer_THT:Potentiometer_Alps_RK09L_Single_Vertical
Connections:
- net +3.3V: now also J1.1 (Pin_1), J1.2 (Pin_2)
- net +5V: now also J1.3 (Pin_3), J1.4 (Pin_4)
- net GND: now also D1.1 (K), D2.1 (K), D3.1 (K), J1.15 (Pin_15), J1.16 (Pin_16), SW1.1
- net MUX_S0: now also J1.8 (Pin_8)
- net MUX_S1: now also J1.9 (Pin_9)
- net MUX_S2: now also J1.10 (Pin_10)
- net SIG_BTN1: now also SW1.2
- net SIG_MUX1: now reaches U1.3 (A)
- net SIG_MUX1: now also J1.5 (Pin_5)
- net SIG_MUX2: now reaches U2.3 (A)
- net SIG_MUX2: now also J1.6 (Pin_6)
- net SIG_MUX3: now reaches U3.3 (A)
- net SIG_MUX3: now also J1.7 (Pin_7)
- new net: D3.2 (A), R3.2
- new net: D2.2 (A), R2.2
- new net: D1.2 (A), R1.2
- new net LED1: J1.11 (Pin_11), R1.1
- new net LED2: J1.12 (Pin_12), R2.1
- new net LED3: J1.13 (Pin_13), R3.1
- no-connect marks 7 -> 5
